File: Wham-Link.kicad_pcb (KiCad board)
At the start: 4 copper layers, 70 x 30 mm, 47 parts, among them J2 Conn_02x05_Counter_Clockwise, J3 Conn_01x09_Pin, SW2 SKRPACE010, SW3 SKRPACE010, U1 LAN8720A-CP-TR, U2 AMS1117-3.3, U3 CH340C, U4 ESP32-WROOM-32UE, X1 ECS-2520MV-250-CN-TR

Commit message: Schematic and layout updates
Parts:
- removed C11: 10uF, Capacitor_SMD:C_0201_0603Metric
- removed C13: 100nF, Capacitor_SMD:C_0402_1005Metric
- moved SW3 28.5 mm to (153.5, 112.7), turned to 0 degrees
- moved R15 22.8 mm to (157.6, 112.8)
- moved C14 21.0 mm to (132.5, 112.8), turned to -90 degrees
- moved C8 20.3 mm to (151.0, 101.1), turned to 0 degrees
- moved C7 18.8 mm to (147.4, 103.2), turned to 0 degrees
- moved R11 18.7 mm to (140.8, 97.3)
- moved R12 18.2 mm to (141.8, 97.3)
- moved C2 16.1 mm to (149.0, 104.5), turned to -90 degrees
- moved R9 14.8 mm to (139.2, 103.8), turned to -90 degrees
- moved R7 14.5 mm to (160.0, 90.2), turned to 180 degrees
- moved R10 14.4 mm to (140.6, 103.8), turned to -90 degrees
- moved C6 14.3 mm to (142.8, 96.5)
- moved R4 14.2 mm to (147.1, 96.6), turned to -90 degrees
- moved R21 13.9 mm to (155.7, 90.3), turned to 180 degrees
- moved R22 13.1 mm to (160.9, 112.6)
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Routing:
- net IO19: track 0.00 -> 43.6 mm, vias 0 -> 2
- net IO5: track 0.00 -> 36.1 mm, vias 0 -> 2
- net IO22: track 0.00 -> 35.5 mm, vias 0 -> 1
- net IO26: track 0.00 -> 31.9 mm, vias 0 -> 2
- net IO18: track 0.00 -> 31.0 mm, vias 0 -> 2
- net IO27: track 0.00 -> 28.2 mm, vias 0 -> 2
- net IO25: track 0.00 -> 27.0 mm
- net IO21: track 0.00 -> 24.8 mm, vias 0 -> 1
- net LED1: track 0.00 -> 23.3 mm, vias 0 -> 2
- net IO23: track 0.00 -> 19.7 mm, vias 0 -> 1
- net LED2: track 0.00 -> 18.3 mm, vias 0 -> 2
- net Net-(U3-D+): track 0.00 -> 14.8 mm, vias 0 -> 2
- net +3V3: track 0.00 -> 14.4 mm
- net Net-(U3-D-): track 0.00 -> 13.4 mm
- net Net-(RJ1-RLED-): track 0.00 -> 13.2 mm
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
Commit message: Schematic and layout updates
Parts:
- moved R15 1.92 mm to (156.7, 111.1)
- moved C12 0.56 mm to (132.9, 107.7)
- moved C9 0.56 mm to (133.9, 107.9)
- moved C15 0.40 mm to (144.8, 89.0)
Routing:
- net RESET: track 0.00 -> 66.9 mm, vias 0 -> 1
- net BOOT: track 0.00 -> 55.5 mm, vias 0 -> 2
- net TXD0: track 0.00 -> 44.6 mm, vias 0 -> 2
- net RXD0: track 0.00 -> 44.0 mm, vias 0 -> 2
- net IO23: track 19.7 -> 45.8 mm, vias 1 -> 2
- net IO22: track 35.5 -> 58.8 mm, vias 1 -> 2
- net IO21: track 24.8 -> 42.6 mm, vias 1 -> 2
- net Net-(U3-V3): track 0.00 -> 15.2 mm, vias 0 -> 2
- net +3V3: track 14.4 -> 29.1 mm
- net GP4: track 0.00 -> 3.96 mm
- net Net-(D4-K): track 0.00 -> 1.61 mm
