File: Wham-Link.kicad_pcb (KiCad board)
At the start: 4 copper layers, 70 x 35 mm, 61 parts, among them J2 Conn_02x05_Counter_Clockwise, J3 Conn_01x09_Pin, Q1 2SC4617R, Q3 UMH3N, SW2 SKRPACE010, SW3 SKRPACE010, U1 LAN8720A-CP-TR, U2 AMS1117-3.3, U3 CH340C, U4 ESP32-WROOM-32UE, X1 ECS-2520MV-250-CN-TR

Commit message: Finish draft layout
Parts:
- moved C10 14.0 mm to (128.7, 105.7)
- moved R18 13.9 mm to (128.6, 104.5), turned to 0 degrees
- moved R13 13.9 mm to (128.6, 103.3), turned to 180 degrees
- moved FB1 11.2 mm to (142.8, 98.5)
- moved TP4 8.90 mm to (156.1, 104.2)
- moved C5 3.59 mm to (141.6, 101.3), turned to 0 degrees
- moved C6 2.22 mm to (139.6, 102.7), turned to 0 degrees
- moved C12 0.31 mm to (155.6, 81.9)
Routing:
- net +3V3: track 81.6 -> 174.3 mm, vias 2 -> 10
- net +5V: track 45.9 -> 99.7 mm, vias 0 -> 6
- net RTS: track 2.17 -> 42.4 mm, vias 0 -> 2
- net IO5: track 3.78 -> 41.4 mm, vias 1 -> 2
- net GPI39: track 0.00 -> 36.4 mm, vias 0 -> 1
- net /VDD1A: track 64.3 -> 30.0 mm, vias 2 -> 3
- net DTR: track 2.17 -> 36.3 mm, vias 0 -> 3
- net BOOT: track 52.3 -> 79.5 mm
- net TXD0: track 0.00 -> 26.5 mm, vias 0 -> 2
- net RXD0: track 0.00 -> 24.8 mm, vias 0 -> 2
- net Net-(RJ1-RLED-): track 4.31 -> 29.0 mm, vias 1 -> 2
- net GPI36: track 0.00 -> 22.6 mm, vias 0 -> 3
- net GPI34: track 0.00 -> 18.3 mm, vias 0 -> 1
- net GPI35: track 0.00 -> 18.1 mm, vias 0 -> 1
- net GP14: track 50.0 -> 64.2 mm, vias 1 -> 3
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