File: ATOS-Bridge-Comms-core.kicad_pcb (KiCad board)
At the start: 4 copper layers, 70 x 35 mm, 61 parts, among them J2 Conn_02x05_Counter_Clockwise, J3 Conn_01x09_Pin, Q1 2SC4617R, Q3 UMH3N, SW2 SKRPACE010, SW3 SKRPACE010, U1 LAN8720A-CP-TR, U2 AMS1117-3.3, U3 CH340C, U4 ESP32-WROOM-32UE, X1 ECS-2520MV-250-CN-TR

Commit message: Post-design review interim changes
Parts:
- added H1: M3, MountingHole:MountingHole_3.2mm_M3, F.Cu at (178.0, 82.0)
- added H2: M3, MountingHole:MountingHole_3.2mm_M3, F.Cu at (118.0, 82.0)
- added kibuzzard-6A57BE6F: G***, kibuzzard-6A57BE6F, F.Cu at (164.7, 91.5)
- moved R15 31.8 mm to (169.8, 112.2)
- moved Q3 30.4 mm to (178.4, 107.2), turned to 90 degrees
- moved SW3 30.0 mm to (173.5, 111.1)
- moved C16 29.3 mm to (177.0, 110.5)
- moved SW2 24.9 mm to (173.7, 107.5), turned to 0 degrees
- moved D7 11.7 mm to (168.1, 110.9), turned to 0 degrees
- moved TP2 8.14 mm to (123.0, 83.0)
- moved TP3 1.90 mm to (168.5, 106.4)
- moved D4 1.78 mm to (163.0, 108.4)
- moved R21 1.77 mm to (165.0, 106.5), turned to 0 degrees
- moved D3 1.75 mm to (166.8, 108.4)
- moved D8 1.67 mm to (118.2, 89.2), turned to 0 degrees
- moved R22 1.36 mm to (162.2, 106.7), turned to 180 degrees
Routing:
- net +3V3: track 174.3 -> 163.9 mm, vias 10 -> 9
- net GND: track 32.3 -> 29.9 mm, vias 99 -> 93
- net Net-(D7-A): track 4.38 -> 2.45 mm
- net GP14: track 64.2 -> 62.4 mm
- net +5V: track 99.7 -> 100.9 mm
- net Net-(D3-K): track 1.62 -> 2.47 mm
- net BOOT: track 79.5 -> 78.7 mm
- net RTS: track 42.4 -> 41.8 mm
- net EN: track 17.2 -> 16.6 mm, vias 2 -> 1
- net DTR: track 36.3 -> 36.2 mm, vias 3 -> 2
Other:
- board size 70 x 35 mm -> 70 x 37 mm

Commit message: Cleaned up the board and fixed issues mentioned in DR-1
Parts:
- removed Q1: 2SC4617R, imported-project-library:SOT-523-3_L1.6-W0.8-P1.00-LS1.6-BR
- removed R1: 332R, Resistor_SMD:R_0402_1005Metric
- removed R23: 4.7k, Resistor_SMD:R_0402_1005Metric
- removed kibuzzard-6A57BE6F: G***, kibuzzard-6A57BE6F
- added C11: 470pF, Capacitor_SMD:C_0603_1608Metric, F.Cu at (138.9, 111.7)
- added C13: 100nF, Capacitor_SMD:C_0402_1005Metric, F.Cu at (159.7, 82.5)
- added C17: 10uF, Capacitor_SMD:C_0603_1608Metric, F.Cu at (159.2, 83.8)
- added G***: LOGO, imported-project-library:abc, F.Cu at (169.9, 82.0)
- added G***: LOGO, imported-project-library:cat, F.Cu at (148.1, 103.0)
- added G***: LOGO, imported-project-library:cat, F.Cu at (117.9, 97.9)
- added G***: LOGO, imported-project-library:cat, F.Cu at (126.2, 110.1)
- added G***: LOGO, imported-project-library:abc, B.Cu at (117.7, 87.9)
- added G***: LOGO, imported-project-library:abc, B.Cu at (148.3, 110.8)
- added G***: LOGO, imported-project-library:abc, B.Cu at (169.7, 81.8)
- added NT1: NetTie_2, NetTie:NetTie-2_SMD_Pad0.5mm, F.Cu at (177.8, 104.6)
- added R24: 10k, Resistor_SMD:R_0402_1005Metric, F.Cu at (131.1, 108.1)
- added R25: 270R, Resistor_SMD:R_0402_1005Metric, F.Cu at (140.6, 88.8)
- added R26: 270R, Resistor_SMD:R_0402_1005Metric, F.Cu at (123.5, 86.6)
- added TP5: TestPoint_Small, TestPoint:TestPoint_Pad_1.0x1.0mm, F.Cu at (137.4, 109.2)
- added TP6: TestPoint_Small, TestPoint:TestPoint_Pad_1.0x1.0mm, F.Cu at (160.8, 113.4)
- added kibuzzard-6A59294C: G***, kibuzzard-6A59294C, B.Cu at (114.9, 95.2)
- added kibuzzard-6A592971: G***, kibuzzard-6A592971, B.Cu at (115.0, 92.7)
- added kibuzzard-6A5929C7: G***, kibuzzard-6A5929C7, B.Cu at (115.0, 97.8)
- added kibuzzard-6A592B5D: G***, kibuzzard-6A592B5D, B.Cu at (115.1, 113.0)
- added kibuzzard-6A592B8C: G***, kibuzzard-6A592B8C, B.Cu at (115.0, 100.3)
- added kibuzzard-6A592B9D: G***, kibuzzard-6A592B9D, B.Cu at (114.9, 102.8)
- added kibuzzard-6A592BBE: G***, kibuzzard-6A592BBE, B.Cu at (114.9, 105.3)
- added kibuzzard-6A592BE1: G***, kibuzzard-6A592BE1, B.Cu at (115.1, 107.8)
- added kibuzzard-6A592BF0: G***, kibuzzard-6A592BF0, B.Cu at (115.0, 110.3)
- added kibuzzard-6A592C3D: G***, kibuzzard-6A592C3D, F.Cu at (178.6, 112.6)
- added kibuzzard-6A592C47: G***, kibuzzard-6A592C47, F.Cu at (179.0, 111.3)
- added kibuzzard-6A592C76: G***, kibuzzard-6A592C76, B.Cu at (181.5, 102.8)
- added kibuzzard-6A592CA3: G***, kibuzzard-6A592CA3, B.Cu at (181.4, 100.2)
- added kibuzzard-6A592CAD: G***, kibuzzard-6A592CAD, B.Cu at (181.4, 97.6)
- added kibuzzard-6A592CC8: G***, kibuzzard-6A592CC8, B.Cu at (170.8, 107.8)
- added kibuzzard-6A592CD3: G***, kibuzzard-6A592CD3, B.Cu at (170.8, 105.4)
- added kibuzzard-6A592CE4: G***, kibuzzard-6A592CE4, B.Cu at (168.1, 102.7)
- added kibuzzard-6A592CF2: G***, kibuzzard-6A592CF2, B.Cu at (168.2, 100.2)
- added kibuzzard-6A592D1D: G***, kibuzzard-6A592D1D, B.Cu at (181.6, 105.3)
- added kibuzzard-6A592D2C: G***, kibuzzard-6A592D2C, B.Cu at (181.6, 108.6)
- added kibuzzard-6A592D3C: G***, kibuzzard-6A592D3C, B.Cu at (168.1, 97.8)
- added kibuzzard-6A5930FC: G***, kibuzzard-6A5930FC, F.Cu at (121.3, 80.8)
- added kibuzzard-6A59312F: G***, kibuzzard-6A59312F, F.Cu at (137.0, 113.6)
- added kibuzzard-6A59314F: G***, kibuzzard-6A59314F, F.Cu at (122.2, 89.0)
- added kibuzzard-6A593210: G***, kibuzzard-6A593210, F.Cu at (153.4, 104.2)
- added kibuzzard-6A59321C: G***, kibuzzard-6A59321C, F.Cu at (163.2, 113.6)
- added kibuzzard-6A593258: G***, kibuzzard-6A593258, F.Cu at (169.2, 108.8)
- C7: value 10uF -> 1uF
- moved C16 29.1 mm to (164.9, 84.0)
- moved R14 8.88 mm to (170.1, 106.6), turned to 90 degrees
- moved C2 3.11 mm to (131.2, 111.4)
- moved X1 2.16 mm to (134.4, 110.8)
- moved C7 0.74 mm to (140.0, 110.6), turned to -45 degrees
- moved TP2 0.45 mm to (122.5, 83.0)
- moved TP1 0.21 mm to (122.0, 87.5)
Connections:
- R4 pad 1: BOOT -> REFCLK0
- RJ1 pad 10: Net-(Q1-C) -> /LED1
- RJ1 pad 11: +3V3 -> Net-(RJ1-RLED+)
- RJ1 pad 12: Net-(RJ1-RLED-) -> /LED2
- RJ1 pad 9: +3V3 -> Net-(RJ1-LLED+)
- U4 pad 25: BOOT -> REFCLK0
Routing:
- net BOOT: track 78.7 -> 9.18 mm, vias 2 -> 0
- net RTS: track 41.8 -> 93.2 mm
- net DTR: track 36.2 -> 80.6 mm
- net EN: track 16.6 -> 60.2 mm, vias 1 -> 4
- net REFCLK0: track 0.00 -> 36.4 mm, vias 0 -> 2
- net /LED1: track 9.92 -> 43.2 mm
- net Net-(Q1-C): track 31.7 -> 0.00 mm
- net /LED2: track 6.72 -> 35.9 mm, vias 0 -> 2
- net Net-(RJ1-RLED-): track 29.0 -> 0.00 mm, vias 2 -> 0
- net Net-(D7-A): track 2.45 -> 14.7 mm
- net +5V: track 100.9 -> 111.8 mm, vias 6 -> 7
- net +3V3: track 163.9 -> 174.2 mm, vias 9 -> 12
- net Net-(D6-A): track 11.8 -> 18.1 mm, vias 4 -> 2
- net Net-(RJ1-LLED+): track 0.00 -> 5.09 mm
- net GND: track 29.9 -> 25.8 mm, vias 93 -> 104
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- removed copper zone on In2.Cu, net Net-(D6-A)
