File: ATOS-Bridge-Comms-core.kicad_pcb (KiCad board)
At the start: 4 copper layers, 70 x 37 mm, 103 parts, among them J2 Conn_02x05_Counter_Clockwise, J3 Conn_01x09_Pin, Q3 UMH3N, SW2 SKRPACE010, SW3 SKRPACE010, U1 LAN8720A-CP-TR, U2 AMS1117-3.3, U3 CH340C, U4 ESP32-WROOM-32UE, X1 ECS-2520MV-250-CN-TR

Commit message: Cleaned up the board and fixed issues mentioned in DR-1
Parts:
- added kibuzzard-6A595918: G***, kibuzzard-6A595918, F.Cu at (160.4, 106.8)
- TP6: footprint TestPoint:TestPoint_Pad_1.0x1.0mm -> TestPoint:TestPoint_Loop_D2.54mm_Drill1.5mm_Beaded
- moved kibuzzard-6A59321C 3.37 mm to (166.6, 113.6)
- moved TP6 2.95 mm to (163.5, 112.2)
- moved kibuzzard-6A593258 0.86 mm to (169.8, 108.1), turned to 0 degrees
Connections:
- J2 pad 5: Net-(D7-A) -> GND
- J2 pad 7: GND -> Net-(D7-A)
Routing:
- net Net-(D6-A): track 18.1 -> 13.8 mm
- net Net-(D7-A): track 14.7 -> 12.7 mm
- net DTR: track 80.6 -> 82.6 mm
- net +3V3: track 174.2 -> 173.3 mm
- net GND: vias 104 -> 103
- added copper zone on F.Cu, net Net-(D6-A)
