File: ATOS-Bridge-Comms-core.kicad_sch (KiCad schematic)
At the start: 69 parts, among them J2 Conn_02x05_Counter_Clockwise, J3 Conn_01x09_Pin, Q3 UMH3N, SW2 SKRPACE010, SW3 SKRPACE010, U1 LAN8720A-CP-TR, U2 AMS1117-3.3, U3 CH340C, U4 ESP32-WROOM-32UE, X1 ECS-2520MV-250-CN-TR

Commit message: Cleaned up the board and fixed issues mentioned in DR-1
Parts:
- C9: symbol Device:C_Polarized_Small -> Device:C_Small
- H1, H2: now not fitted
- TP6: footprint TestPoint:TestPoint_Pad_1.0x1.0mm -> TestPoint:TestPoint_Loop_D2.54mm_Drill1.5mm_Beaded; LCSC Part (none) -> C5199801; now fitted
Connections:
- net GND: now also J2.5 (Pin_5); no longer J2.7 (Pin_7)
- net at D7.2 (A): now also J2.7 (Pin_7); no longer J2.5 (Pin_5)
Other:
- moved on the sheet: D7
Changed lines of the file:
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@@
 	(wire
 		(pts
-			(xy 143.51 191.77) (xy 148.59 191.77)
-		)
-		(stroke
-			(width 0)
-			(type default)
-		)
-	)
-	(wire
-		(pts
 			(xy 219.71 44.45) (xy 220.98 44.45)
 		)
@@
 	(wire
 		(pts
+			(xy 137.16 191.77) (xy 148.59 191.77)
+		)
+		(stroke
+			(width 0)
+			(type default)
+		)
+	)
+	(wire
+		(pts
 			(xy 59.69 144.78) (xy 59.69 147.32)
 		)
@@
 	(wire
 		(pts
+			(xy 172.72 177.8) (xy 172.72 189.23)
+		)
+		(stroke
+			(width 0)
+			(type default)
+		)
+	)
+	(wire
+		(pts
 			(xy 93.98 124.46) (xy 93.98 127)
 		)
@@
 	(wire
 		(pts
-			(xy 135.89 191.77) (xy 138.43 191.77)
+			(xy 135.89 177.8) (xy 162.56 177.8)
 		)
 		(stroke
@@
 	(wire
 		(pts
-			(xy 161.29 189.23) (xy 172.72 189.23)
-		)
-		(stroke
-			(width 0)
-			(type default)
-		)
-	)
-	(wire
-		(pts
 			(xy 142.24 175.26) (xy 137.16 175.26)
 		)
@@
 	(wire
 		(pts
-			(xy 135.89 191.77) (xy 135.89 175.26)
+			(xy 172.72 189.23) (xy 161.29 189.23)
+		)
+		(stroke
+			(width 0)
+			(type default)
+		)
+	)
+	(wire
+		(pts
+			(xy 135.89 177.8) (xy 135.89 175.26)
 		)
 		(stroke
@@
 	(wire
 		(pts
+			(xy 167.64 177.8) (xy 172.72 177.8)
+		)
+		(stroke
+			(width 0)
+			(type default)
+		)
+	)
+	(wire
+		(pts
 			(xy 135.89 171.45) (xy 135.89 170.18)
 		)
@@
 		(on_board yes)
 		(in_pos_files yes)
-		(dnp no)
+		(dnp yes)
 		(fields_autoplaced yes)
 		(property "Reference" "H2"
@@
 	)
 	(symbol
-		(lib_id "Device:C_Polarized_Small")
+		(lib_id "Device:C_Small")
 		(at 102.87 110.49 270)
 		(unit 1)
@@
 		(fields_autoplaced yes)
 		(property "Reference" "C9"
-			(at 103.4161 104.14 90)
+			(at 102.8636 104.14 90)
 			(show_name no)
 			(do_not_autoplace no)
@@
 		)
 		(property "Value" "10uF"
-			(at 103.4161 106.68 90)
+			(at 102.8636 106.68 90)
 			(show_name no)
 			(do_not_autoplace no)
@@
 			)
 		)
-		(property "Description" "Polarized capacitor, small symbol"
+		(property "Description" "Unpolarized capacitor, small symbol"
 			(at 102.87 110.49 0)
 			(hide yes)
@@
 	(symbol
 		(lib_id "Device:D_Small_Filled")
-		(at 140.97 191.77 0)
+		(at 165.1 177.8 0)
 		(unit 1)
 		(body_style 1)
@@
 		(dnp no)
 		(property "Reference" "D7"
-			(at 139.954 193.294 0)
+			(at 164.084 179.324 0)
 			(show_name no)
 			(do_not_autoplace no)
@@
 		)
 		(property "Value" "D_Small_Filled"
-			(at 139.7001 194.31 90)
+			(at 163.8301 180.34 90)
 			(hide yes)
 			(show_name no)
@@
 		)
 		(property "Footprint" "imported-project-library:DIO-SMD_L2.0-W1.9-LS3.8-RD"
-			(at 140.97 191.77 90)
+			(at 165.1 177.8 90)
 			(hide yes)
 			(show_name no)
@@
 		)
 		(property "Datasheet" ""
-			(at 140.97 191.77 90)
+			(at 165.1 177.8 90)
 			(hide yes)
 			(show_name no)
@@
 		)
 		(property "Description" "Diode, small symbol, filled shape"
-			(at 140.97 191.77 0)
+			(at 165.1 177.8 0)
 			(hide yes)
 			(show_name no)
@@
 		)
 		(property "Sim.Device" "D"
-			(at 140.97 191.77 0)
+			(at 165.1 177.8 0)
 			(hide yes)
 			(show_name no)
@@
 		)
 		(property "Sim.Pins" "1=K 2=A"
-			(at 140.97 191.77 0)
+			(at 165.1 177.8 0)
 			(hide yes)
 			(show_name no)
@@
 		(on_board yes)
 		(in_pos_files yes)
-		(dnp no)
+		(dnp yes)
 		(fields_autoplaced yes)
 		(property "Reference" "H1"
@@
 		(on_board yes)
 		(in_pos_files yes)
-		(dnp yes)
+		(dnp no)
 		(property "Reference" "TP6"
-			(at 33.02 179.07 0)
+			(at 28.448 180.34 0)
 			(show_name no)
 			(do_not_autoplace no)
@@
 			)
 		)
-		(property "Footprint" "TestPoint:TestPoint_Pad_1.0x1.0mm"
+		(property "Footprint" "TestPoint:TestPoint_Loop_D2.54mm_Drill1.5mm_Beaded"
 			(at 38.1 180.34 0)
 			(hide yes)
@@
 			)
 		)
+		(property "LCSC Part" "C5199801"
+			(at 33.02 180.34 0)
+			(hide yes)
+			(show_name no)
+			(do_not_autoplace no)
+			(effects
+				(font
+					(size 1.27 1.27)
+				)
+			)
+		)
 		(pin "1"
 		)
@@
 	(symbol
 		(lib_id "power:GND")
-		(at 172.72 189.23 0)
+		(at 137.16 191.77 0)
 		(mirror y)
 		(unit 1)
@@
 		(dnp no)
 		(property "Reference" "#PWR053"
-			(at 172.72 195.58 0)
+			(at 137.16 198.12 0)
 			(hide yes)
 			(show_name no)
@@
 		)
 		(property "Value" "GND"
-			(at 172.212 188.468 0)
+			(at 136.652 191.008 0)
 			(show_name no)
 			(do_not_autoplace no)
@@
 		)
 		(property "Footprint" ""
-			(at 172.72 189.23 0)
+			(at 137.16 191.77 0)
 			(hide yes)
 			(show_name no)
@@
 		)
 		(property "Datasheet" ""
-			(at 172.72 189.23 0)
+			(at 137.16 191.77 0)
 			(hide yes)
 			(show_name no)
@@
 		)
 		(property "Description" "Power symbol creates a global label with name \"GND\" , ground"
-			(at 172.72 189.23 0)
+			(at 137.16 191.77 0)
 			(hide yes)
 			(show_name no)
